File: Power Regulators.sch (KiCad schematic (older format))
At the start: 21 parts, among them J4 CONN_02JST-PTH-2, Q2 DMG2305UX-13, Q5 DMG2305UX-13, U3 MCP73811T-420I-OT, U5 AP2112K-3.3, U6 MAX1704X

Commit message: Replace USB to UART with CP2102-GM
Parts:
- U5: DigiKey(Alt) (none) -> https://www.digikey.com/en/products/detail/diodes-incorpora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
Changed lines of the file:
@@
 F 2 "Package_TO_SOT_SMD:SOT-23-5" H 8445 2775 50  0001 C CNN
 F 3 "https://www.diodes.com/assets/Datasheets/AP2112.pdf" H 8445 2550 50  0001 C CNN
+F 4 "https://www.digikey.com/en/products/detail/diodes-incorporated/AP7365-33WG-7/4249847" H 8445 2450 50  0001 C CNN "DigiKey(Alt)"
 	1    8445 2450
 	1    0    0    -1

Commit message: Update board
Parts:
- removed U3: MCP73811T-420I-OT, Package_TO_SOT_SMD:SOT-23-5, symbol Battery_Management:MCP73811T-420I-OT
- added U3: MCP73832-2-OT, Package_TO_SOT_SMD:SOT-23-5, symbol Battery_Management:MCP73832-2-OT
Connections:
- net +3V3: no longer S1.1
- net +BATT: now also U3.3 (VBAT)
- net +VUSB_IN: now also U3.4 (VDD)
- net GND: now also U3.2 (VSS)
- net V_PREMOS: now reaches D3.1 (K), Q2.2 (S), Q5.2 (S)
- net V_PREMOS: now also S1.1
- net at R9.1: now also U3.5 (PROG)
Changed lines of the file:
@@
-$EndComp
-$Comp
-L Battery_Management:MCP73811T-420I-OT U?
-U 1 1 60DC1181
-P 6575 5245
-AR Path="/60DC1181" Ref="U?"  Part="1"
-AR Path="/60D841D7/60DC1181" Ref="U3"  Part="1"
-F 0 "U3" H 6275 5495 50  0000 L CNN
-F 1 "MCP73811T-420I-OT" H 6325 4495 50  0000 L CNN
-F 2 "Package_TO_SOT_SMD:SOT-23-5" H 6625 4995 50  0001 L CNN
-F 3 "http://ww1.microchip.com/downloads/en/DeviceDoc/22036b.pdf" H 6325 5495 50  0001 C CNN
-	1    6575 5245
-	1    0    0    -1
 $EndComp
 $Comp
@@
 	1    0    0    -1
 $EndComp
-NoConn ~ 6175 5145
-Wire Wire Line
-	6575 4795 6575 4945
 $Comp
 L power:GND #PWR?
@@
 L power:GND #PWR?
 U 1 1 60DC1195
-P 6575 5645
+P 6600 5650
 AR Path="/60DC1195" Ref="#PWR?"  Part="1"
 AR Path="/60D841D7/60DC1195" Ref="#PWR0125"  Part="1"
-F 0 "#PWR0125" H 6575 5395 50  0001 C CNN
-F 1 "GND" H 6580 5472 50  0000 C CNN
-F 2 "" H 6575 5645 50  0001 C CNN
-F 3 "" H 6575 5645 50  0001 C CNN
-	1    6575 5645
-	1    0    0    -1
-$EndComp
-Wire Wire Line
-	6575 5645 6575 5545
+F 0 "#PWR0125" H 6600 5400 50  0001 C CNN
+F 1 "GND" H 6605 5477 50  0000 C CNN
+F 2 "" H 6600 5650 50  0001 C CNN
+F 3 "" H 6600 5650 50  0001 C CNN
+	1    6600 5650
+	1    0    0    -1
+$EndComp
 Wire Wire Line
 	5675 5345 5675 5445
@@
 $EndComp
 Wire Wire Line
-	6175 5345 6075 5345
-Wire Wire Line
 	6075 5345 6075 5395
 $Comp
@@
 Wire Wire Line
 	7325 4895 7325 5145
-Wire Wire Line
-	7325 5145 6975 5145
 $Comp
 L Device:C C?
@@
 L MiOrigin:+VUSB_IN #PWR0137
 U 1 1 60DF442D
-P 6575 4795
-F 0 "#PWR0137" H 6575 4645 50  0001 C CNN
-F 1 "+VUSB_IN" H 6590 4968 50  0000 C CNN
-F 2 "" H 6575 4795 50  0001 C CNN
-F 3 "" H 6575 4795 50  0001 C CNN
-	1    6575 4795
+P 6600 4765
+F 0 "#PWR0137" H 6600 4615 50  0001 C CNN
+F 1 "+VUSB_IN" H 6615 4938 50  0000 C CNN
+F 2 "" H 6600 4765 50  0001 C CNN
+F 3 "" H 6600 4765 50  0001 C CNN
+	1    6600 4765
 	1    0    0    -1
 $EndComp
@@
 $EndComp
 Wire Wire Line
-	7020 2350 6770 2350
-Text GLabel 7095 2700 0    50   Input ~ 0
+	7020 2350 6895 2350
+Text GLabel 7145 2700 2    50   Input ~ 0
 EN_SWITCH
 Wire Wire Line
-	7095 2700 7120 2700
+	7145 2700 7120 2700
 Wire Wire Line
 	7120 2700 7120 2650
@@
 	0    1    1    0
 $EndComp
-$Comp
-L power:+3.3V #PWR0140
-U 1 1 60DF5E20
-P 5280 7050
-F 0 "#PWR0140" H 5280 6900 50  0001 C CNN
-F 1 "+3.3V" H 5295 7223 50  0000 C CNN
-F 2 "" H 5280 7050 50  0001 C CNN
-F 3 "" H 5280 7050 50  0001 C CNN
-	1    5280 7050
-	1    0    0    -1
-$EndComp
-Wire Wire Line
-	5280 7050 5280 7110
 Wire Wire Line
 	5280 7110 5320 7110
@@
 Wire Wire Line
 	5420 1600 5420 2000
+NoConn ~ 7000 5345
+Wire Wire Line
+	6600 5545 6600 5650
+Wire Wire Line
+	6600 4945 6600 4765
+Wire Wire Line
+	7325 5145 7000 5145
+$Comp
+L Battery_Management:MCP73832-2-OT U3
+U 1 1 60D60955
+P 6600 5245
+F 0 "U3" H 6450 5640 50  0000 C CNN
+F 1 "MCP73832-2-OT" H 6225 5555 50  0000 C CNN
+F 2 "Package_TO_SOT_SMD:SOT-23-5" H 6650 4995 50  0001 L CIN
+F 3 "http://ww1.microchip.com/downloads/en/DeviceDoc/20001984g.pdf" H 6450 5195 50  0001 C CNN
+F 4 "https://www.digikey.com/en/products/detail/microchip-technology/MCP73832T-2DCI-OT/1223150" H 6600 5245 50  0001 C CNN "DigiKey"
+	1    6600 5245
+	1    0    0    -1
+$EndComp
+Wire Wire Line
+	6075 5345 6200 5345
+Text GLabel 6870 2775 0    50   Input ~ 0
+V_PREMOS
+Connection ~ 6895 2350
+Wire Wire Line
+	6895 2350 6770 2350
+Text GLabel 5100 6850 0    50   Input ~ 0
+V_PREMOS
+Wire Wire Line
+	5280 6850 5100 6850
+Wire Wire Line
+	5280 6850 5280 7110
+Wire Wire Line
+	6870 2775 6895 2775
+Wire Wire Line
+	6895 2350 6895 2775
 $EndSCHEMATC
