File: pcb/Power Regulators.sch (KiCad schematic (older format))
At the start: 21 parts, among them J4 CONN_02JST-PTH-2, Q2 DMG2305UX-13, Q5 DMG2305UX-13, U3 MCP73832-2-OT, U5 AP2112K-3.3, U6 MAX1704X

Commit message: Few updates
Other:
- moved on the sheet: C8, U6
Changed lines of the file:
@@
 encoding utf-8
 Sheet 3 3
-Title ""
-Date ""
-Rev ""
-Comp ""
-Comment1 ""
+Title "MiOrigin Controller"
+Date "2021-06-11"
+Rev "1.1"
+Comp "Aerosol Technologies Lab - BAEN @ TAMU"
+Comment1 "Author: Charlemagne Wong | CECN 21'"
 Comment2 ""
 Comment3 ""
@@
 L SparkFun-IC-Power:MAX1704X U?
 U 1 1 60D9F7EA
-P 1720 5890
+P 1755 4055
 AR Path="/60D9F7EA" Ref="U?"  Part="1"
 AR Path="/60D841D7/60D9F7EA" Ref="U6"  Part="1"
-F 0 "U6" H 1720 6450 45  0000 C CNN
-F 1 "MAX1704X" H 1720 6366 45  0000 C CNN
-F 2 "MAX17048G_T10:SON50P200X200X80-9N" H 1720 6290 20  0001 C CNN
-F 3 "" H 1720 5890 60  0001 C CNN
-F 4 "IC-10399" H 1720 6271 60  0000 C CNN "Field4"
-F 5 "https://www.digikey.com/en/products/detail/maxim-integrated/MAX17048G-T10/3758921" H 1720 5890 50  0001 C CNN "DigiKey"
-F 6 "MAX17048G+T10" H 1720 5890 50  0001 C CNN "MPN"
-	1    1720 5890
-	1    0    0    -1
-$EndComp
-Text GLabel 2670 5690 2    50   Input ~ 0
+F 0 "U6" H 1755 4615 45  0000 C CNN
+F 1 "MAX1704X" H 1755 4531 45  0000 C CNN
+F 2 "MAX17048G_T10:SON50P200X200X80-9N" H 1755 4455 20  0001 C CNN
+F 3 "" H 1755 4055 60  0001 C CNN
+F 4 "IC-10399" H 1755 4436 60  0000 C CNN "Field4"
+F 5 "https://www.digikey.com/en/products/detail/maxim-integrated/MAX17048G-T10/3758921" H 1755 4055 50  0001 C CNN "DigiKey"
+F 6 "MAX17048G+T10" H 1755 4055 50  0001 C CNN "MPN"
+	1    1755 4055
+	1    0    0    -1
+$EndComp
+Text GLabel 2705 3855 2    50   Input ~ 0
 SDA
-Text GLabel 2670 5790 2    50   Input ~ 0
+Text GLabel 2705 3955 2    50   Input ~ 0
 SCL
 $Comp
 L power:GND #PWR?
 U 1 1 60D9F7F5
-P 1070 6190
+P 1105 4355
 AR Path="/60D9F7F5" Ref="#PWR?"  Part="1"
 AR Path="/60D841D7/60D9F7F5" Ref="#PWR0119"  Part="1"
-F 0 "#PWR0119" H 1070 5940 50  0001 C CNN
-F 1 "GND" H 1075 6017 50  0000 C CNN
-F 2 "" H 1070 6190 50  0001 C CNN
-F 3 "" H 1070 6190 50  0001 C CNN
-	1    1070 6190
-	1    0    0    -1
-$EndComp
-Wire Wire Line
-	1070 6190 1070 6090
-Wire Wire Line
-	1070 5990 1220 5990
-Wire Wire Line
-	1220 6090 1070 6090
-Connection ~ 1070 6090
-Wire Wire Line
-	1070 6090 1070 5990
-Wire Wire Line
-	1070 5990 1070 5690
-Wire Wire Line
-	1070 5690 1220 5690
-Connection ~ 1070 5990
-Wire Wire Line
-	1120 5590 1120 5790
-Wire Wire Line
-	1120 5890 1220 5890
-Wire Wire Line
-	1220 5790 1120 5790
-Connection ~ 1120 5790
-Wire Wire Line
-	1120 5790 1120 5890
+F 0 "#PWR0119" H 1105 4105 50  0001 C CNN
+F 1 "GND" H 1110 4182 50  0000 C CNN
+F 2 "" H 1105 4355 50  0001 C CNN
+F 3 "" H 1105 4355 50  0001 C CNN
+	1    1105 4355
+	1    0    0    -1
+$EndComp
+Wire Wire Line
+	1105 4355 1105 4255
+Wire Wire Line
+	1105 4155 1255 4155
+Wire Wire Line
+	1255 4255 1105 4255
+Connection ~ 1105 4255
+Wire Wire Line
+	1105 4255 1105 4155
+Wire Wire Line
+	1105 4155 1105 3855
+Wire Wire Line
+	1105 3855 1255 3855
+Connection ~ 1105 4155
+Wire Wire Line
+	1155 3755 1155 3955
+Wire Wire Line
+	1155 4055 1255 4055
+Wire Wire Line
+	1255 3955 1155 3955
+Connection ~ 1155 3955
+Wire Wire Line
+	1155 3955 1155 4055
 $Comp
 L power:GND #PWR?
 U 1 1 60D9F809
-P 2320 6190
+P 2355 4355
 AR Path="/60D9F809" Ref="#PWR?"  Part="1"
 AR Path="/60D841D7/60D9F809" Ref="#PWR0120"  Part="1"
-F 0 "#PWR0120" H 2320 5940 50  0001 C CNN
-F 1 "GND" H 2325 6017 50  0000 C CNN
-F 2 "" H 2320 6190 50  0001 C CNN
-F 3 "" H 2320 6190 50  0001 C CNN
-	1    2320 6190
-	1    0    0    -1
-$EndComp
-Wire Wire Line
-	2320 6190 2320 5890
-Wire Wire Line
-	2320 5890 2220 5890
+F 0 "#PWR0120" H 2355 4105 50  0001 C CNN
+F 1 "GND" H 2360 4182 50  0000 C CNN
+F 2 "" H 2355 4355 50  0001 C CNN
+F 3 "" H 2355 4355 50  0001 C CNN
+	1    2355 4355
+	1    0    0    -1
+$EndComp
+Wire Wire Line
+	2355 4355 2355 4055
+Wire Wire Line
+	2355 4055 2255 4055
 $Comp
 L power:+BATT #PWR?
 U 1 1 60D9F817
-P 2730 6360
+P 2765 4525
 AR Path="/60D9F817" Ref="#PWR?"  Part="1"
 AR Path="/60D841D7/60D9F817" Ref="#PWR0121"  Part="1"
-F 0 "#PWR0121" H 2730 6210 50  0001 C CNN
-F 1 "+BATT" H 2745 6533 50  0000 C CNN
-F 2 "" H 2730 6360 50  0001 C CNN
-F 3 "" H 2730 6360 50  0001 C CNN
-	1    2730 6360
+F 0 "#PWR0121" H 2765 4375 50  0001 C CNN
+F 1 "+BATT" H 2780 4698 50  0000 C CNN
+F 2 "" H 2765 4525 50  0001 C CNN
+F 3 "" H 2765 4525 50  0001 C CNN
+	1    2765 4525
 	1    0    0    -1
 $EndComp
@@
 L power:GND #PWR?
 U 1 1 60D9F81F
-P 2730 6740
+P 2765 4905
 AR Path="/60D9F81F" Ref="#PWR?"  Part="1"
 AR Path="/60D841D7/60D9F81F" Ref="#PWR0122"  Part="1"
-F 0 "#PWR0122" H 2730 6490 50  0001 C CNN
-F 1 "GND" H 2735 6567 50  0000 C CNN
-F 2 "" H 2730 6740 50  0001 C CNN
-F 3 "" H 2730 6740 50  0001 C CNN
-	1    2730 6740
-	1    0    0    -1
-$EndComp
-Text Notes 2150 4800 2    118  ~ 0
+F 0 "#PWR0122" H 2765 4655 50  0001 C CNN
+F 1 "GND" H 2770 4732 50  0000 C CNN
+F 2 "" H 2765 4905 50  0001 C CNN
+F 3 "" H 2765 4905 50  0001 C CNN
+	1    2765 4905
+	1    0    0    -1
+$EndComp
+Text Notes 2390 3080 2    118  ~ 0
 Fuel Gauge
 $Comp
 L power:+BATT #PWR?
 U 1 1 60D9F82F
-P 1120 5590
+P 1155 3755
 AR Path="/60D9F82F" Ref="#PWR?"  Part="1"
 AR Path="/60D841D7/60D9F82F" Ref="#PWR0123"  Part="1"
-F 0 "#PWR0123" H 1120 5440 50  0001 C CNN
-F 1 "+BATT" H 1135 5763 50  0000 C CNN
-F 2 "" H 1120 5590 50  0001 C CNN
-F 3 "" H 1120 5590 50  0001 C CNN
-	1    1120 5590
+F 0 "#PWR0123" H 1155 3605 50  0001 C CNN
+F 1 "+BATT" H 1170 3928 50  0000 C CNN
+F 2 "" H 1155 3755 50  0001 C CNN
+F 3 "" H 1155 3755 50  0001 C CNN
+	1    1155 3755
 	1    0    0    -1
 $EndComp
@@
 L Device:C C?
 U 1 1 60D9F811
-P 2730 6550
+P 2765 4715
 AR Path="/60D9F811" Ref="C?"  Part="1"
 AR Path="/60D841D7/60D9F811" Ref="C8"  Part="1"
-F 0 "C8" H 2550 6500 50  0000 C CNN
-F 1 "0.1uF" H 2490 6600 50  0000 C CNN
-F 2 "Capacitor_SMD:C_0603_1608Metric" H 2768 6400 50  0001 C CNN
-F 3 "" H 2730 6550 50  0001 C CNN
-F 4 "https://www.digikey.com/en/products/detail/kemet/C0603C104J4RACTU/411096" H 2730 6550 50  0001 C CNN "DigiKey"
-	1    2730 6550
+F 0 "C8" H 2585 4665 50  0000 C CNN
+F 1 "0.1uF" H 2525 4765 50  0000 C CNN
+F 2 "Capacitor_SMD:C_0603_1608Metric" H 2803 4565 50  0001 C CNN
+F 3 "" H 2765 4715 50  0001 C CNN
+F 4 "https://www.digikey.com/en/products/detail/kemet/C0603C104J4RACTU/411096" H 2765 4715 50  0001 C CNN "DigiKey"
+	1    2765 4715
 	-1   0    0    1
 $EndComp
 Wire Wire Line
-	2730 6700 2730 6740
-Wire Wire Line
-	2730 6360 2730 6400
+	2765 4865 2765 4905
+Wire Wire Line
+	2765 4525 2765 4565
 Wire Notes Line
 	6970 6540 3430 6540
@@
 	3430 470  3430 7790
 Wire Notes Line
-	470  4330 3430 4330
-Wire Notes Line
 	3430 3510 11220 3510
 Wire Wire Line
-	2220 5690 2670 5690
-Wire Wire Line
-	2220 5790 2670 5790
-Text GLabel 2670 5990 2    50   Input ~ 0
+	2255 3855 2705 3855
+Wire Wire Line
+	2255 3955 2705 3955
+Text GLabel 2705 4155 2    50   Input ~ 0
 BAT_ALERT
 Wire Wire Line
-	2220 5990 2670 5990
+	2255 4155 2705 4155
 $Comp
 L Connector:TestPoint TP3
