File: pcb/USB.sch (KiCad schematic (older format))
At the start: 14 parts, among them J2 USB_C_Receptacle, U2 CP2102

Commit message: Few updates
Other:
- note added: "USB to UART"
- note added: "USB-C ESD Protection TVS Diode"
- moved on the sheet: C1, C10, C18, C19, D1, U2
